File: ESP32C3.kicad_pcb (KiCad board)
At the start: 2 copper layers, 50 x 55 mm, 42 parts, among them J1 USB_C_Receptacle_USB2.0, J2 Conn_01x04, SW1 NST, SW2 BOOT, U1 USBLC6-2SC6-SOT236, U2 Crystal4, U3 ESP32-C3, U4 TLV1117-33

Commit message: maybe finish.
Parts:
- added J3: Conn_01x18, Connector_PinHeader_2.54mm:PinHeader_1x18_P2.54mm_Vertical, F.Cu at (84.7, 32.9)
- added J4: Conn_01x18, Connector_PinSocket_2.54mm:PinSocket_1x18_P2.54mm_Vertical, F.Cu at (89.3, 32.9)
- AE1: footprint RF_Antenna:Texas_SWRA117D_2.4GHz_Left -> RF_Antenna:Texas_SWRA117D_2.4GHz_Right
- moved SW2 49.5 mm to (77.7, 32.4)
- moved C15 43.9 mm to (78.0, 38.0), turned to 180 degrees
- moved REF** 43.4 mm to (69.5, 74.4)
- moved R10 42.3 mm to (78.0, 39.6), turned to 0 degrees
- moved R6 33.3 mm to (80.5, 40.1), turned to 90 degrees
- moved R7 16.2 mm to (80.5, 69.0), turned to -90 degrees
- moved SW1 13.7 mm to (81.2, 82.2), turned to 180 degrees
- moved L1 9.43 mm to (54.5, 75.1)
- moved AE1 9.38 mm to (54.5, 79.1)
- moved C2 8.12 mm to (55.3, 72.7)
- moved C1 7.82 mm to (55.3, 77.4)
- moved C9 3.68 mm to (73.2, 64.1)
- moved R1 2.50 mm to (73.7, 38.7)
- moved R2 2.50 mm to (75.4, 38.7)
- moved R9 2.16 mm to (72.1, 82.9)
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Routing:
- net VDD3P3_CPU: track 14.3 -> 195.0 mm, vias 0 -> 5
- net BOOT: track 0.00 -> 50.1 mm, vias 0 -> 1
- net /GPIO8: track 0.00 -> 39.0 mm, vias 0 -> 1
- net /U0_RX: track 0.00 -> 36.5 mm, vias 0 -> 2
- net /GPIO10: track 0.00 -> 35.9 mm
- net /GPIO5: track 0.00 -> 34.3 mm
- net /GPIO2: track 0.00 -> 34.0 mm, vias 0 -> 2
- net Net-(R4-Pad1): track 0.00 -> 33.7 mm, vias 0 -> 2
- net /GPIO0: track 0.00 -> 32.3 mm
- net /GPIO7: track 0.00 -> 31.7 mm
- net /GPIO6: track 0.00 -> 30.2 mm
- net /GPIO1: track 0.00 -> 29.7 mm
- net /GPIO4: track 0.00 -> 28.4 mm
- net EN: track 0.00 -> 28.1 mm, vias 0 -> 2
- net /GPIO3: track 0.00 -> 27.1 mm
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- added copper zone on B.Cu, net GND
- added copper zone on F.Cu, net GND
