File: ESP32C3.kicad_sch (KiCad schematic)
At the start: 30 parts

Commit message: Made some changes.
Parts:
- removed C? (x2): 22p, symbol Device:C_Small
- removed C? (x2): 0.1u, symbol Device:C_Small
- removed D?: 1N5819, Diode_THT:D_DO-41_SOD81_P10.16mm_Horizontal, symbol Diode:1N5819
- removed R?: 10k, symbol Device:R
- removed SW?: boot, symbol Switch:SW_Push
- removed Y?: 40M, symbol Device:Crystal_GND24
- added AE?: Antenna_Chip, symbol Device:Antenna_Chip
- added C? (x2): 0.1u, symbol Device:C_Small
- added C? (x2): 22p, symbol Device:C_Small
- added C?: 1u, symbol Device:C_Small
- added D?: LED, symbol Device:LED
- added D?: D_TVS_Filled, symbol Device:D_TVS_Filled
- added F?: Fuse_Small, symbol Device:Fuse_Small
- added J?: Conn_01x04, symbol Connector_Generic:Conn_01x04
- added R? (x2): 22R, symbol Device:R
- added R?: 470, symbol Device:R
- added R?: 10k, symbol Device:R
- added SW?: BOOT, symbol Switch:SW_Push
- added U?: USBLC6-2SC6-SOT236, symbol Library:USBLC6-2SC6-SOT236
- added U?: Crystal4, symbol Library:Crystal4
- SW?: value nst -> NST
Connections:
- net +3.3V: now also C?.1, C?.1, J?.1 (Pin_1), R?.1, R?.1
- net +5V: now also D?.2 (A2), F?.2, U?.5 (VCC)
- net GND: now also AE?.2 (PCB_Trace), C?.2, C?.2, C?.2, C?.2, C?.2, D?.1 (A1), D?.1 (K), J?.4 (Pin_4), SW?.1, U?.2, U?.2 (GND), U?.4
- net USB_DN: now also R?.2; no longer J?.A7 (D-), J?.B7 (D-)
- net USB_DP: now also R?.2; no longer J?.A6 (D+), J?.B6 (D+)
- net at U?.30 (XTAL_P): now also C?.1, U?.3
- net at U?.29 (XTAL_N): now also C?.1, U?.1
- net BOOT: now reaches U?.15 (GPIO9/BOOT)
- net BOOT: now also C?.1, R?.2, SW?.2
- net GPIO8: now reaches R?.1, U?.14 (GPIO8)
- net VDD3P3: now reaches C?.1, L?.2, U?.2 (VDD3P3), U?.3 (VDD3P3)
- net GPIO2: now reaches R?.1, U?.6 (GPIO2/ADC1_CH2)
- net GPIO12: no longer names the net of U?.19 (SPIHD/GPIO12)
- net GPIO13: no longer names the net of U?.20 (SPIWP/GPIO13)
- net GPIO14: no longer names the net of U?.21 (SPICS0/GPIO14)
- net GPIO15: no longer names the net of U?.22 (SPICLK/GPIO15)
- net GPIO16: no longer names the net of U?.23 (SPID/GPIO16)
- net GPIO17: no longer names the net of U?.24 (SPIQ/GPIO17)
- net LNA: no longer names the net of C?.1, L?.1
- net LNA: now also AE?.1 (FEED)
- net Uart_RX renamed U0_RX
- net U0_RX: now also J?.3 (Pin_3)
- net Uart_TX renamed U0_TX
- net U0_TX: now also J?.2 (Pin_2)
- net VBUS: no longer names the net of J?.A4 (VBUS), J?.A9 (VBUS), J?.B4 (VBUS), J?.B9 (VBUS)
- net VBUS: now also F?.1
- new net: D?.2 (A), R?.2
- new net: R?.1, U?.4 (I/O2)
- new net: J?.A7 (D-), J?.B7 (D-), U?.1 (I/O1)
- new net: J?.A6 (D+), J?.B6 (D+), U?.3 (I/O2)
- new net: R?.1, U?.6 (I/O1)
- no-connect marks 2 -> 8
Other:
- moved on the sheet: C?, L?, R?, SW?, U?

Commit message: Changes.
Parts:
- added D3: LED, LED_SMD:LED_0603_1608Metric, symbol Device:LED
- added R11: 470, Resistor_SMD:R_0603_1608Metric, symbol Device:R
- AE1: renamed from AE?; footprint (none) -> RF_Antenna:Texas_SWRA117D_2.4GHz_Left
- C1, C10, C11, C12, C13, C14, C15, C2, C3, C4, C7, C8, C9: renamed from C?; footprint (none) -> Capacitor_SMD:C_0603_1608Metric
- C5, C6: renamed from C?; footprint (none) -> Capacitor_SMD:C_0805_2012Metric
- D1: renamed from D?; footprint (none) -> Library:X1-DFN1006-2_L1.0-W0.6-BI
- D2: renamed from D?; footprint (none) -> LED_SMD:LED_0603_1608Metric
- F1: renamed from F?; footprint (none) -> Fuse:Fuse_1206_3216Metric
- J1: renamed from J?; footprint (none) -> Connector_USB:USB_C_Receptacle_XKB_U262-16XN-4BVC11
- J2: renamed from J?; footprint (none) -> Connector_Harwin:Harwin_M20-89004xx_1x04_P2.54mm_Horizontal
- L1: renamed from L?; footprint (none) -> Inductor_SMD:L_0603_1608Metric
- L2: renamed from L?; footprint (none) -> Inductor_SMD:L_0805_2012Metric
- R1, R10, R2, R3, R4, R5, R6, R7, R8, R9: renamed from R?; footprint (none) -> Resistor_SMD:R_0603_1608Metric
- SW1, SW2: renamed from SW?; footprint (none) -> Library:SW-SMD_L6.0-W3.3-LS8.0
- U1: renamed from U?; footprint (none) -> Package_TO_SOT_SMD:SOT-23-6
- U2: renamed from U?; footprint (none) -> Crystal:Crystal_SMD_3225-4Pin_3.2x2.5mm
- U4: renamed from U?; footprint (none) -> Package_TO_SOT_SMD:SOT-223-3_TabPin2
- gave numbers to parts that had none: 1
Connections:
- net +3.3V: now also R11.1
- net GPIO11: now also D3.1 (K)
- new net: D3.2 (A), R11.2
Other:
- moved on the sheet: D1

Commit message: maybe finish.
Parts:
- added J3: Conn_01x18, Connector_PinHeader_2.54mm:PinHeader_1x18_P2.54mm_Vertical, symbol Connector_Generic:Conn_01x18
- added J4: Conn_01x18, Connector_PinSocket_2.54mm:PinSocket_1x18_P2.54mm_Vertical, symbol Connector_Generic:Conn_01x18
- AE1: footprint RF_Antenna:Texas_SWRA117D_2.4GHz_Left -> RF_Antenna:Texas_SWRA117D_2.4GHz_Right
Connections:
- net +3.3V: now also J3.10 (Pin_10), J3.18 (Pin_18), J3.2 (Pin_2), J4.10 (Pin_10), J4.18 (Pin_18), J4.2 (Pin_2)
- net BOOT: now also J3.4 (Pin_4), J4.4 (Pin_4)
- net GND: now also J3.1 (Pin_1), J3.16 (Pin_16), J3.17 (Pin_17), J3.9 (Pin_9), J4.1 (Pin_1), J4.16 (Pin_16), J4.17 (Pin_17), J4.9 (Pin_9)
- net GPIO0: now also J3.15 (Pin_15), J4.15 (Pin_15)
- net GPIO1: now also J3.14 (Pin_14), J4.14 (Pin_14)
- net GPIO10: now also J3.3 (Pin_3), J4.3 (Pin_3)
- net GPIO2: now also J3.13 (Pin_13), J4.13 (Pin_13)
- net GPIO3: now also J3.12 (Pin_12), J4.12 (Pin_12)
- net GPIO4: now also J3.11 (Pin_11), J4.11 (Pin_11)
- net GPIO5: now also J3.8 (Pin_8), J4.8 (Pin_8)
- net GPIO6: now also J3.7 (Pin_7), J4.7 (Pin_7)
- net GPIO7: now also J3.6 (Pin_6), J4.6 (Pin_6)
- net GPIO8: now also J3.5 (Pin_5), J4.5 (Pin_5)
